Commit message: 首次提交代码

File: robot_description/water_description/urdf/depthcam.xacro (robot description, xacro)
@@ -109,5 +109,5 @@
       <enable_wind>0</enable_wind>
       <kinematic>0</kinematic>
-      <gravity>1</gravity>
+      <gravity>true</gravity>
       <mu2>1</mu2>
       <fdir1>0 0 0</fdir1>

File: robot_description/water_description/urdf/water_all.xacro (robot description, xacro)
@@ -5,4 +5,10 @@
 <robot name="water_all" xmlns:xacro="http://ros.org/wiki/xacro">
   <xacro:property name="M_PI" value="3.1415926535897931" />
+  <link name="base_footprint"/>
+  <joint name="base_footprint_joint" type="fixed">
+    <parent link="base_footprint"/>
+    <child link="base_link"/>
+    <origin xyz="0 0 0" rpy="0 0 0"/>
+  </joint>
   <link
     name="base_link">
@@ -38,9 +44,8 @@
     <collision>
       <origin
-        xyz="0 0 0"
-        rpy="0 0 0" />
-      <geometry>
-        <mesh
-          filename="package://water_description/meshes/base_link.STL" />
+        xyz="0 0 0.04"
+        rpy="0 0 -${M_PI/2}" />
+      <geometry>
+        <cylinder length="0.15" radius="0.26"/>
       </geometry>
     </collision>
@@ -76,37 +81,37 @@
     <parent link="base_link2"/>
     <child link="wheel_left_link"/>
+    <origin xyz="-${0.40/2} 0.0 -0.04" rpy="${-M_PI/2} 0 ${M_PI/2}"/>
+    <axis xyz="0 0 1"/>
+  </joint>
+  <link name="wheel_left_link">
+    <visual>
+      <material
+        name="">
+        <color
+          rgba="1.0 1.0 1.0 1" />
+      </material>
+      <geometry>
+        <cylinder length="0.0206" radius="0.028"/>
+      </geometry>
+      <origin xyz="0 0 0" rpy="0 0 0"/>
+    </visual>
+    <collision>
+      <geometry>
+        <cylinder length="0.0206" radius="0.028"/>
+      </geometry>
+      <origin rpy="0 0 0" xyz="0 0 0"/>
+    </collision>
+    <inertial>
+      <mass value="0.01" />
+      <origin xyz="0 0 0" />
+      <inertia ixx="0.001" ixy="0.0" ixz="0.0"
+                iyy="0.001" iyz="0.0"
+                izz="0.001" />
+    </inertial>
+  </link>
+  <joint name="wheel_right_joint" type="continuous">
+    <parent link="base_link2"/>
+    <child link="wheel_right_link"/>
     <origin xyz="${0.40/2} 0.0 -0.04" rpy="${-M_PI/2} 0 ${M_PI/2}"/>
-    <axis xyz="0 0 1"/>
-  </joint>
-  <link name="wheel_left_link">
-    <visual>
-      <material
-        name="">
-        <color
-          rgba="1.0 1.0 1.0 1" />
-      </material>
-      <geometry>
-        <cylinder length="0.0206" radius="0.028"/>
-      </geometry>
-      <origin xyz="0 0 0" rpy="0 0 0"/>
-    </visual>
-    <collision>
-      <geometry>
-        <cylinder length="0.0206" radius="0.028"/>
-      </geometry>
-      <origin rpy="0 0 0" xyz="0 0 0"/>
-    </collision>
-    <inertial>
-      <mass value="0.01" />
-      <origin xyz="0 0 0" />
-      <inertia ixx="0.001" ixy="0.0" ixz="0.0"
-                iyy="0.001" iyz="0.0"
-                izz="0.001" />
-    </inertial>
-  </link>
-  <joint name="wheel_right_joint" type="continuous">
-    <parent link="base_link2"/>
-    <child link="wheel_right_link"/>
-    <origin xyz="-${0.40/2} 0.0 -0.04" rpy="${-M_PI/2} 0 ${M_PI/2}"/>
     <axis xyz="0 0 1"/>
   </joint>
@@ -356,10 +361,10 @@
   <!-- Hokuyo Laser -->
   <link name="hokuyo_link">
-    <collision>
+    <!-- <collision>
       <origin xyz="0 0 0" rpy="0 0 0"/>
       <geometry>
         <box size="0.01 0.01 0.01"/>
       </geometry>
-    </collision>
+    </collision> -->
     <visual>
       <origin xyz="0 0 0" rpy="0 0 0"/>
@@ -427,11 +432,18 @@
       <rightJoint>wheel_right_joint</rightJoint>
       <wheelSeparation>0.40</wheelSeparation>
-      <wheelDiameter>0.03</wheelDiameter>
-      <torque>300</torque>
+      <wheelDiameter>0.056</wheelDiameter>
+      <wheelTorque>300</wheelTorque>
+      <wheelAcceleration>1.0</wheelAcceleration>
+      <rosDebugLevel>na</rosDebugLevel>
+      <publishWheelJointState>true</publishWheelJointState>
+      <odometrySource>world</odometrySource>
+      <publishTf>1</publishTf>
       <legacyMode>true</legacyMode>
       <commandTopic>cmd_vel</commandTopic>
       <odometryTopic>odom</odometryTopic>
       <odometryFrame>odom</odometryFrame>
-      <robotBaseFrame>base_link</robotBaseFrame>
+      <robotBaseFrame>base_footprint</robotBaseFrame>
+      <publishWheelTF>true</publishWheelTF>
+      <publishOdomTF>true</publishOdomTF>
     </plugin>
   </gazebo>
@@ -466,7 +478,16 @@
       <plugin name="gazebo_ros_head_hokuyo_controller" filename="libgazebo_ros_laser.so">
         <topicName>/scan</topicName>
-        <frameName>base_link</frameName>
+        <frameName>hokuyo_link</frameName>
       </plugin>
     </sensor>
   </gazebo>
+  <gazebo reference="base_link">
+    <collision name="base_link_collision">
+      <surface>
+        <contact>
+          <collide_bitmask>0x02</collide_bitmask>
+        </contact>
+      </surface>
+    </collision>
+  </gazebo>
 </robot>

File: robot_description/wheeltec_description/urdf/mini_akm/miniakm_transmission.xacro (robot description, xacro)
@@ -44,5 +44,5 @@
   <gazebo>
     <plugin name="gazebo_ros_control" filename="libgazebo_ros_control.so">
-      <robotNamespace>/wheeltec</robotNamespace>
+      <!-- <robotNamespace>/wheeltec</robotNamespace> -->
       <robotSimType>gazebo_ros_control/DefaultRobotHWSim</robotSimType>
     </plugin>
